Commit message: update filling

File: linorobot2_description/urdf/mecanum_properties.urdf.xacro (robot description, xacro)
@@ -1,15 +1,16 @@
 <?xml version="1.0"?>
 <robot xmlns:xacro="http://ros.org/wiki/xacro">
-  <xacro:property name="base_length" value="0.445" />
-  <xacro:property name="base_width" value="0.200" />
+  <xacro:property name="base_length" value="0.5" />
+  <xacro:property name="base_width" value="0.5" />
   <xacro:property name="base_height" value="0.129" />
   <xacro:property name="base_mass" value="10" />
   <xacro:property name="wheel_radius" value="0.07162" />
   <xacro:property name="wheel_width" value="0.05" />
-  <xacro:property name="wheel_pos_x" value="0.120" />
-  <xacro:property name="wheel_pos_y" value="0.1355" />
+  <xacro:property name="wheel_pos_x" value="0.25" />
+  <xacro:property name="wheel_pos_y" value="0.25" />
   <xacro:property name="wheel_pos_z" value="-0.04788" />
   <xacro:property name="wheel_mass" value=".6" />
   <xacro:property name="wheel_torque" value="20" />
+  <xacro:property name="wheel_yaw" value = "0.785398163"/>
   <xacro:property name="laser_pose">
     <origin xyz="-0.0475 0 0.125" rpy="0 0 0"/>

File: linorobot2_description/urdf/mech/mecanum_wheel.urdf.xacro (robot description, xacro)
@@ -1,5 +1,5 @@
 <?xml version="1.0"?>
 <robot xmlns:xacro="http://ros.org/wiki/xacro">
-  <xacro:macro name="mecanum_wheel" params="side radius width pos_x pos_y pos_z mass">
+  <xacro:macro name="mecanum_wheel" params="side radius width pos_x pos_y pos_z mass yaw">
     <link name="${side}_wheel_link">
       <visual>
@@ -44,5 +44,5 @@
       <parent link="base_link"/>
       <child link="${side}_wheel_link"/>
-      <origin xyz="${pos_x} ${pos_y} ${pos_z}" rpy="0 0 0"/>
+      <origin xyz="${pos_x} ${pos_y} ${pos_z}" rpy="0 0 ${yaw}"/>
     </joint>
   </xacro:macro>

File: linorobot2_description/urdf/robots/mecanum.urdf.xacro (robot description, xacro)
@@ -24,4 +24,5 @@
     pos_z="${wheel_pos_z}"
     mass="${wheel_mass}"
+    yaw = "${-wheel_yaw}"
   />
   <xacro:mecanum_wheel
@@ -33,4 +34,5 @@
     pos_z="${wheel_pos_z}"
     mass="${wheel_mass}"
+    yaw = "${wheel_yaw}"
   />
   <xacro:mecanum_wheel
@@ -42,4 +44,5 @@
     pos_z="${wheel_pos_z}"
     mass="${wheel_mass}"
+    yaw = "${wheel_yaw}"
   />
   <xacro:mecanum_wheel
@@ -51,4 +54,5 @@
     pos_z="${wheel_pos_z}"
     mass="${wheel_mass}"
+    yaw = "${-wheel_yaw}"
   />
   <xacro:imu/>
